Commit message: feat(driver): add FrRobotHardwareInterface and the real-hardware launch
The real-hardware plugin, on the client library (software version
3.8.4). read() and write() never touch the network: read() takes the
newest state frame without waiting and reports a stale frame, a lost
link or a broken servo stream as a communication fault (ERROR, ->
unconfigured); a robot fault, emergency stop or safety stop halts the
stream and deactivates. Faults are never cleared automatically: the
operator calls ~/reset_error, which uses its own XML-RPC connection
and is refused during an emergency stop or a communication fault. A
command that asks for more than one step limit (URDF velocity limit *
cmdT) is refused before the firmware sees it. Deactivating flushes the
firmware queue with STOP first. ServoJ goes through ServoSender with
the drift compensation and the idle pause fed from the state frames.

The connections are created once in on_init and only connected and
disconnected by the lifecycle callbacks, so the service thread never
sees one replaced; the shutdown work of on_deactivate/on_error, which
run on the realtime thread, happens on a cleanup thread that catches
any exception. The launch file starts the real hardware inactive and
activates it as a separate step, so a failed precondition leaves the
controller manager and ~/reset_error running. The tests drive the
plugin through the ResourceManager against a fake controller.

Assisted-by: pi/claude-opus-5-5
Assisted-by: pi/claude-sonnet-5-5

File: fr_robot_driver/urdf/fr_controlled.urdf.xacro (robot description, xacro)
@@ -10,4 +10,7 @@
       use_mock_hardware      : mock_components/GenericSystem (default true)
       initial_positions_file : ros2_control initial positions
+      ip, cmd_t_ms, prefill, update_rate_hz, namespace, allow_unverified_version:
+                             real hardware only, see fr_ros2_control.xacro
+      mock_gpio_commands     : mock only, loop-back command interfaces on fr_status
   -->
   <xacro:arg name="model" default="fairino20_v6"/>
@@ -16,4 +19,11 @@
   <xacro:arg name="initial_positions_file"
              default="$(find fr_robot_driver)/config/initial_positions.yaml"/>
+  <xacro:arg name="mock_gpio_commands" default="false"/>
+  <xacro:arg name="ip" default="192.168.58.2"/>
+  <xacro:arg name="cmd_t_ms" default="8"/>
+  <xacro:arg name="prefill" default="3"/>
+  <xacro:arg name="update_rate_hz" default="125"/>
+  <xacro:arg name="namespace" default=""/>
+  <xacro:arg name="allow_unverified_version" default="false"/>
   <xacro:include filename="$(find fr_description)/urdf/fr_macro.xacro"/>
   <xacro:include filename="$(find fr_robot_driver)/urdf/fr_ros2_control.xacro"/>
@@ -28,4 +38,11 @@
       tf_prefix="${tf_prefix}"
       use_mock_hardware="$(arg use_mock_hardware)"
+      mock_gpio_commands="$(arg mock_gpio_commands)"
+      ip="$(arg ip)"
+      cmd_t_ms="$(arg cmd_t_ms)"
+      prefill="$(arg prefill)"
+      update_rate_hz="$(arg update_rate_hz)"
+      namespace="$(arg namespace)"
+      allow_unverified_version="$(arg allow_unverified_version)"
       initial_positions_file="$(arg initial_positions_file)"/>
 </robot>

File: fr_robot_driver/urdf/fr_ros2_control.xacro (robot description, xacro)
@@ -18,6 +18,14 @@
       initial_positions_file  : YAML with initial_positions map (unprefixed joint names)
       mock_sensor_commands    : mock GPIO sensor commands (default false)
-    The real-hardware branch is a placeholder: the fr_robot_driver hardware
-    plugin will be filled in once the mock pipeline is validated end to end.
+    Both branches expose the same <gpio name="<tf_prefix>fr_status"> state interfaces
+    (docs/fault_handling.md section 7). With the mock, mock_gpio_commands:=true adds command
+    interfaces that loop back into them, to rehearse fault handling in upper layers.
+    Real hardware (fr_robot_driver/FrRobotHardwareInterface) parameters:
+      ip                         : controller address (default 192.168.58.2)
+      cmd_t_ms / prefill         : ServoJ cmdT in whole ms (default 8) / standing segments at start (3)
+      update_rate_hz             : controller_manager update rate; update_rate_hz * cmd_t_ms / 1000
+                                   must be an integer >= 1 (default 1000 / cmd_t_ms)
+      namespace                  : namespace of the reset_error service node
+      allow_unverified_version   : run against a software version that is not whitelisted (default false)
   -->
   <!-- Internal helper: one ros2_control joint (name prefixed like the URDF joints).
@@ -36,8 +44,31 @@
     </joint>
   </xacro:macro>
+  <!-- Internal helper: the fr_status gpio, identical for mock and real hardware. -->
+  <xacro:macro name="_fr_status_gpio" params="tf_prefix">
+    <gpio name="${tf_prefix}fr_status">
+      <state_interface name="fault_class"><param name="initial_value">0.0</param></state_interface>
+      <state_interface name="estop"><param name="initial_value">0.0</param></state_interface>
+      <state_interface name="safety_stop0"><param name="initial_value">0.0</param></state_interface>
+      <state_interface name="safety_stop1"><param name="initial_value">0.0</param></state_interface>
+      <state_interface name="collision"><param name="initial_value">0.0</param></state_interface>
+      <state_interface name="main_code"><param name="initial_value">0.0</param></state_interface>
+      <state_interface name="sub_code"><param name="initial_value">0.0</param></state_interface>
+      <state_interface name="enabled"><param name="initial_value">1.0</param></state_interface>
+      <state_interface name="robot_mode"><param name="initial_value">0.0</param></state_interface>
+      <state_interface name="robot_state"><param name="initial_value">1.0</param></state_interface>
+      <state_interface name="servo_queue_len"><param name="initial_value">0.0</param></state_interface>
+    </gpio>
+  </xacro:macro>
   <xacro:macro name="fr_ros2_control" params="
       tf_prefix:=''
       use_mock_hardware:=true
       mock_sensor_commands:='false'
+      mock_gpio_commands:='false'
+      ip:='192.168.58.2'
+      cmd_t_ms:=8
+      prefill:=3
+      update_rate_hz:=125
+      namespace:=''
+      allow_unverified_version:='false'
       initial_positions_file">
     <xacro:property name="initial_positions"
@@ -48,10 +79,15 @@
           <plugin>mock_components/GenericSystem</plugin>
           <param name="mock_sensor_commands">${mock_sensor_commands}</param>
+          <param name="mock_gpio_commands">${mock_gpio_commands}</param>
         </xacro:if>
         <xacro:unless value="${use_mock_hardware}">
-          <!-- placeholder: real Fairino hardware plugin (progressive development:
-               enabled once the mock pipeline below is validated) -->
           <plugin>fr_robot_driver/FrRobotHardwareInterface</plugin>
           <param name="tf_prefix">${tf_prefix}</param>
+          <param name="ip">${ip}</param>
+          <param name="cmd_t_ms">${cmd_t_ms}</param>
+          <param name="prefill">${prefill}</param>
+          <param name="update_rate_hz">${update_rate_hz}</param>
+          <param name="namespace">${namespace}</param>
+          <param name="allow_unverified_version">${allow_unverified_version}</param>
         </xacro:unless>
       </hardware>
@@ -68,4 +104,5 @@
       <xacro:_fr_hw_joint joint_name="wrist_3_joint" tf_prefix="${tf_prefix}"
           initial_position="${initial_positions['wrist_3_joint']}"/>
+      <xacro:_fr_status_gpio tf_prefix="${tf_prefix}"/>
     </ros2_control>
   </xacro:macro>

Commit message: feat(driver): check the controller model and flange pose against FK
The URDF (limits, kinematics) is built for one model, so configure
refuses a controller of another model, and an unknown one unless
allow_unknown_model is set. Configure and activate also compare the
state frame's flange pose with the forward kinematics of its joint
angles (fr_description parameters passed in by xacro), which catches
wrong zero offsets, sign conventions or installation; the deviation is
logged when the check passes (fk_check:=false disables it).

Assisted-by: pi/claude-opus-5-5

File: fr_robot_driver/urdf/fr_controlled.urdf.xacro (robot description, xacro)
@@ -10,5 +10,6 @@
       use_mock_hardware      : mock_components/GenericSystem (default true)
       initial_positions_file : ros2_control initial positions
-      ip, cmd_t_ms, prefill, update_rate_hz, namespace, allow_unverified_version:
+      ip, cmd_t_ms, prefill, update_rate_hz, namespace, allow_unverified_version,
+      allow_unknown_model, fk_check, fk_position_tolerance_mm, fk_angle_tolerance_deg:
                              real hardware only, see fr_ros2_control.xacro
       mock_gpio_commands     : mock only, loop-back command interfaces on fr_status
@@ -26,4 +27,8 @@
   <xacro:arg name="namespace" default=""/>
   <xacro:arg name="allow_unverified_version" default="false"/>
+  <xacro:arg name="allow_unknown_model" default="false"/>
+  <xacro:arg name="fk_check" default="true"/>
+  <xacro:arg name="fk_position_tolerance_mm" default="10.0"/>
+  <xacro:arg name="fk_angle_tolerance_deg" default="1.0"/>
   <xacro:include filename="$(find fr_description)/urdf/fr_macro.xacro"/>
   <xacro:include filename="$(find fr_robot_driver)/urdf/fr_ros2_control.xacro"/>
@@ -45,4 +50,10 @@
       namespace="$(arg namespace)"
       allow_unverified_version="$(arg allow_unverified_version)"
+      model="$(arg model)"
+      kinematics_parameters_file="$(find fr_description)/config/$(arg model)/default_kinematics.yaml"
+      allow_unknown_model="$(arg allow_unknown_model)"
+      fk_check="$(arg fk_check)"
+      fk_position_tolerance_mm="$(arg fk_position_tolerance_mm)"
+      fk_angle_tolerance_deg="$(arg fk_angle_tolerance_deg)"
       initial_positions_file="$(arg initial_positions_file)"/>
 </robot>

File: fr_robot_driver/urdf/fr_ros2_control.xacro (robot description, xacro)
@@ -28,4 +28,10 @@
       namespace                  : namespace of the reset_error service node
       allow_unverified_version   : run against a software version that is not whitelisted (default false)
+      model                      : fr_description model this URDF was built for (fairino5_v6, ...); the
+                                   controller's model string must match it, or configure fails
+      kinematics_parameters_file : that model's default_kinematics.yaml; the plugin cross-checks the
+                                   state frame's flange_cur_pos against its own FK of the joint angles
+      allow_unknown_model, fk_check, fk_position_tolerance_mm, fk_angle_tolerance_deg:
+                                   tuning of the two checks, see fr_robot_driver/README.md
   -->
   <!-- Internal helper: one ros2_control joint (name prefixed like the URDF joints).
@@ -71,4 +77,10 @@
       namespace:=''
       allow_unverified_version:='false'
+      model:=''
+      kinematics_parameters_file:=''
+      allow_unknown_model:='false'
+      fk_check:='true'
+      fk_position_tolerance_mm:=10.0
+      fk_angle_tolerance_deg:=1.0
       initial_positions_file">
     <xacro:property name="initial_positions"
@@ -90,4 +102,13 @@
           <param name="namespace">${namespace}</param>
           <param name="allow_unverified_version">${allow_unverified_version}</param>
+          <param name="model">${model}</param>
+          <param name="allow_unknown_model">${allow_unknown_model}</param>
+          <param name="fk_check">${fk_check}</param>
+          <param name="fk_position_tolerance_mm">${fk_position_tolerance_mm}</param>
+          <param name="fk_angle_tolerance_deg">${fk_angle_tolerance_deg}</param>
+          <!-- joint origins "x y z r p y" per joint, in joint order, plus the flange offset -->
+          <xacro:property name="kin" value="${xacro.load_yaml(kinematics_parameters_file)}"/>
+          <param name="kinematics">${';'.join([kin['kinematics'][j]['xyz'] + ' ' + kin['kinematics'][j]['rpy'] for j in ['shoulder_pan_joint', 'shoulder_lift_joint', 'elbow_joint', 'wrist_1_joint', 'wrist_2_joint', 'wrist_3_joint']])}</param>
+          <param name="flange_offset">${kin['flange_offset']}</param>
         </xacro:unless>
       </hardware>

Commit message: feat(driver): PGI-140 gripper through ros2_control
gripper:=pgi140 mounts the gripper on tool0 and adds the joint
left_finger_joint (opening 0-0.04 m) with gripper_controller
(parallel_gripper_action_controller); mock and real hardware share the
interface. On real hardware:

- ~/gripper/activate is the only way to activate (it always opens to
  the full stroke); refused while active, with a robot fault, while the
  arm moves or is streamed to
- commands are passed on only from a gripper_controller started on a
  usable gripper, so an old goal never runs after an activation or a
  fault; MoveGripper goes out through GripperSender, only when the
  newest opening differs and the servo stream has paused (the
  controller holds MoveGripper back while ServoJ flows, G8)
- while the gripper moves, an arm command that would move is refused
  and the arm held (the controller would queue the ServoJ, G9), until
  the frame shows the motion done, none within 1.5 s, or 30 s; a failed
  MoveGripper call is judged by the frame too, as the controller may
  still run it. Once the gripper is done the command has 2 s to return
  to where the arm stands, otherwise the driver makes a protective stop
  (the step check's stop is the other kind; the reason is in
  ~/status). joint_trajectory_controller gets a path tolerance of
  0.26 rad so that a held trajectory aborts early
- the opening comes from the frame, held during a motion while the
  frame says 0 %, and fully open after an activation or while not
  active (the widest outline for collision checks)

The README states that arm and gripper should not be commanded at the
same time. The gripper plan with its real-robot results and the
measurements G8-G11 and S18 come along.

Assisted-by: pi/claude-opus-5-5

File: fr_robot_driver/urdf/fr_controlled.urdf.xacro (robot description, xacro)
@@ -14,4 +14,7 @@
                              real hardware only, see fr_ros2_control.xacro
       mock_gpio_commands     : mock only, a loop-back command interface on fr_status/fault_class
+      gripper                : end effector on tool0: none (default) or pgi140
+                               (gripper_dahuan_pgi140, one more joint in ros2_control)
+      gripper_index          : real hardware only, the controller's gripper number (default 1)
   -->
   <xacro:arg name="model" default="fairino20_v6"/>
@@ -32,7 +35,13 @@
   <xacro:arg name="fk_position_tolerance_mm" default="10.0"/>
   <xacro:arg name="fk_angle_tolerance_deg" default="1.0"/>
+  <xacro:arg name="gripper" default="none"/>
+  <xacro:arg name="gripper_index" default="1"/>
   <xacro:include filename="$(find fr_description)/urdf/fr_macro.xacro"/>
   <xacro:include filename="$(find fr_robot_driver)/urdf/fr_ros2_control.xacro"/>
   <xacro:property name="tf_prefix" value="$(arg tf_prefix)"/>
+  <xacro:property name="gripper" value="$(arg gripper)"/>
+  <xacro:if value="${gripper not in ['none', 'pgi140']}">
+    ${xacro.fatal("gripper must be none or pgi140, not '" + gripper + "'")}
+  </xacro:if>
   <xacro:fr_robot
       tf_prefix="${tf_prefix}"
@@ -41,6 +50,12 @@
       physical_parameters_file="$(find fr_description)/config/$(arg model)/physical_parameters.yaml"
       visual_parameters_file="$(find fr_description)/config/$(arg model)/visual_parameters.yaml"/>
+  <xacro:if value="${gripper == 'pgi140'}">
+    <xacro:include filename="$(find gripper_dahuan_pgi140)/urdf/gripper_dahuan_pgi140_macro.xacro"/>
+    <xacro:gripper_dahuan_pgi140 tf_prefix="${tf_prefix}" parent="tool0"/>
+  </xacro:if>
   <xacro:fr_ros2_control
       tf_prefix="${tf_prefix}"
+      gripper="${gripper}"
+      gripper_index="$(arg gripper_index)"
       use_mock_hardware="$(arg use_mock_hardware)"
       mock_gpio_commands="$(arg mock_gpio_commands)"

File: fr_robot_driver/urdf/fr_ros2_control.xacro (robot description, xacro)
@@ -18,4 +18,8 @@
       initial_positions_file  : YAML with initial_positions map (unprefixed joint names)
       mock_sensor_commands    : mock GPIO sensor commands (default false)
+      gripper                 : none (default) or pgi140: adds the joint <tf_prefix>left_finger_joint
+                                (gripper_dahuan_pgi140) with commands position [m], max_velocity
+                                [m/s], max_effort [N] and states position, velocity
+      gripper_index           : real hardware only, the controller's gripper number (default 1)
     Both branches expose the same <gpio name="<tf_prefix>fr_status"> with one state interface,
     fault_class (docs/fault_handling.md section 7). With the mock, mock_gpio_commands:=true adds a
@@ -51,4 +55,27 @@
     </joint>
   </xacro:macro>
+  <!-- Internal helper: the gripper joint, identical for mock and real hardware. The joint limiter
+       stays off: it would turn a jump of the opening into a ramp of separate gripper commands; the
+       plugin clamps the opening to the stroke itself. -->
+  <xacro:macro name="_fr_gripper_joint" params="tf_prefix">
+    <joint name="${tf_prefix}left_finger_joint">
+      <limits enable="false"/>
+      <command_interface name="position">
+        <param name="initial_value">0.0</param>
+      </command_interface>
+      <command_interface name="max_velocity">
+        <param name="initial_value">0.0</param>
+      </command_interface>
+      <command_interface name="max_effort">
+        <param name="initial_value">0.0</param>
+      </command_interface>
+      <state_interface name="position">
+        <param name="initial_value">0.0</param>
+      </state_interface>
+      <state_interface name="velocity">
+        <param name="initial_value">0.0</param>
+      </state_interface>
+    </joint>
+  </xacro:macro>
   <!-- Internal helper: the fr_status gpio, identical for mock and real hardware. -->
   <xacro:macro name="_fr_status_gpio" params="tf_prefix">
@@ -75,4 +102,6 @@
       fk_position_tolerance_mm:=10.0
       fk_angle_tolerance_deg:=1.0
+      gripper:='none'
+      gripper_index:=1
       initial_positions_file">
     <xacro:property name="initial_positions"
@@ -104,4 +133,8 @@
           <param name="kinematics">${';'.join([kin['kinematics'][j]['xyz'] + ' ' + kin['kinematics'][j]['rpy'] for j in ['shoulder_pan_joint', 'shoulder_lift_joint', 'elbow_joint', 'wrist_1_joint', 'wrist_2_joint', 'wrist_3_joint']])}</param>
           <param name="flange_offset">${kin['flange_offset']}</param>
+          <xacro:if value="${gripper != 'none'}">
+            <param name="gripper_joint">${tf_prefix}left_finger_joint</param>
+            <param name="gripper_index">${gripper_index}</param>
+          </xacro:if>
         </xacro:unless>
       </hardware>
@@ -118,4 +151,7 @@
       <xacro:_fr_hw_joint joint_name="wrist_3_joint" tf_prefix="${tf_prefix}"
           initial_position="${initial_positions['wrist_3_joint']}"/>
+      <xacro:if value="${gripper != 'none'}">
+        <xacro:_fr_gripper_joint tf_prefix="${tf_prefix}"/>
+      </xacro:if>
       <xacro:_fr_status_gpio tf_prefix="${tf_prefix}"/>
     </ros2_control>

Commit message: feat(driver): pause trajectories while the gripper is busy
The hardware exports <tf_prefix>speed_scaling/speed_scaling_factor, as
the UR driver does, and joint_trajectory_controller uses it: 1.0
normally, 0.0 on real hardware while the gripper moves or activates.
A trajectory then waits where it is instead of running ahead of an arm
that the controller does not move during a gripper motion. The mock
keeps 1.0.

Assisted-by: pi/claude-opus-5-5

File: fr_robot_driver/urdf/fr_controlled.urdf.xacro (robot description, xacro)
@@ -13,5 +13,5 @@
       allow_unknown_model, fk_check, fk_position_tolerance_mm, fk_angle_tolerance_deg:
                              real hardware only, see fr_ros2_control.xacro
-      mock_gpio_commands     : mock only, a loop-back command interface on fr_status/fault_class
+      mock_gpio_commands     : mock only, loop-back command interfaces on fr_status/fault_class and speed_scaling/speed_scaling_factor
       gripper                : end effector on tool0: none (default) or pgi140
                                (gripper_dahuan_pgi140, one more joint in ros2_control)

File: fr_robot_driver/urdf/fr_ros2_control.xacro (robot description, xacro)
@@ -23,6 +23,9 @@
       gripper_index           : real hardware only, the controller's gripper number (default 1)
     Both branches expose the same <gpio name="<tf_prefix>fr_status"> with one state interface,
-    fault_class (docs/fault_handling.md section 7). With the mock, mock_gpio_commands:=true adds a
-    command interface that loops back into it, to rehearse fault handling in upper layers.
+    fault_class (docs/fault_handling.md section 7), and <gpio name="<tf_prefix>speed_scaling"> with
+    speed_scaling_factor, the joint_trajectory_controller's speed scaling (as ur_robot_driver): 1.0,
+    and 0.0 on real hardware while the gripper is busy, so a trajectory waits instead of running
+    ahead of an arm that cannot move (sdk_quirks G9). With the mock, mock_gpio_commands:=true adds
+    command interfaces that loop back into both, to rehearse fault handling and pauses in upper layers.
     Real hardware (fr_robot_driver/FrRobotHardwareInterface) parameters:
       ip                         : controller address (default 192.168.58.2)
@@ -82,4 +85,10 @@
     <gpio name="${tf_prefix}fr_status">
       <state_interface name="fault_class"><param name="initial_value">0.0</param></state_interface>
+    </gpio>
+  </xacro:macro>
+  <!-- Internal helper: the speed_scaling gpio, identical for mock and real hardware. -->
+  <xacro:macro name="_fr_speed_scaling_gpio" params="tf_prefix">
+    <gpio name="${tf_prefix}speed_scaling">
+      <state_interface name="speed_scaling_factor"><param name="initial_value">1.0</param></state_interface>
     </gpio>
   </xacro:macro>
@@ -155,4 +164,5 @@
       </xacro:if>
       <xacro:_fr_status_gpio tf_prefix="${tf_prefix}"/>
+      <xacro:_fr_speed_scaling_gpio tf_prefix="${tf_prefix}"/>
     </ros2_control>
   </xacro:macro>
