Commit message: refactor(description): declare gripper command interfaces on mock only
On real hardware the plugin provides the gripper action itself and sends
MoveGripper over XML-RPC; it never reads the left_finger_joint command
interfaces. Declaring them invited a controller to claim them and write
values that did nothing. They now exist only on mock hardware, where the
upstream parallel_gripper_action_controller writes them; the state
interfaces stay everywhere for joint_states and TF.

Assisted-by: pi/claude-opus-5-5

File: fr_robot_driver/urdf/fr_ros2_control.xacro (robot description, xacro)
@@ -19,5 +19,7 @@
       mock_sensor_commands    : mock GPIO sensor commands (default false)
       gripper                 : none (default) or pgi140: adds the joint <tf_prefix>left_finger_joint
-                                (gripper_dahuan_pgi140) with commands position [m], max_effort [N]
+                                (gripper_dahuan_pgi140) with the opening as a state interface;
+                                mock hardware also gets the position and max_effort command
+                                interfaces the upstream gripper controller writes
                                 and states position, velocity
       gripper_index           : real hardware only, the controller's gripper number (default 1)
@@ -58,16 +60,22 @@
     </joint>
   </xacro:macro>
-  <!-- Internal helper: the gripper joint, identical for mock and real hardware. The joint limiter
-       stays off: it would turn a jump of the opening into a ramp of separate gripper commands; the
-       plugin clamps the opening to the stroke itself. -->
-  <xacro:macro name="_fr_gripper_joint" params="tf_prefix">
+  <!-- Internal helper: the gripper joint. The opening is a state interface everywhere, so it
+       reaches joint_states and TF. Its command interfaces exist on mock hardware only: the mock's
+       parallel_gripper_action_controller writes them, while on real hardware the plugin serves the
+       same action itself and moves the gripper over its own XML-RPC channel (the driver never reads
+       these interfaces; declaring them there would invite a controller that does nothing). The joint
+       limiter stays off: it would turn a jump of the opening into a ramp of separate gripper
+       commands; the plugin clamps the opening to the stroke itself. -->
+  <xacro:macro name="_fr_gripper_joint" params="tf_prefix mock">
     <joint name="${tf_prefix}left_finger_joint">
       <limits enable="false"/>
-      <command_interface name="position">
-        <param name="initial_value">0.0</param>
-      </command_interface>
-      <command_interface name="max_effort">
-        <param name="initial_value">0.0</param>
-      </command_interface>
+      <xacro:if value="${mock}">
+        <command_interface name="position">
+          <param name="initial_value">0.0</param>
+        </command_interface>
+        <command_interface name="max_effort">
+          <param name="initial_value">0.0</param>
+        </command_interface>
+      </xacro:if>
       <state_interface name="position">
         <param name="initial_value">0.0</param>
@@ -158,5 +166,5 @@
           initial_position="${initial_positions['wrist_3_joint']}"/>
       <xacro:if value="${gripper != 'none'}">
-        <xacro:_fr_gripper_joint tf_prefix="${tf_prefix}"/>
+        <xacro:_fr_gripper_joint tf_prefix="${tf_prefix}" mock="${use_mock_hardware}"/>
       </xacro:if>
       <xacro:_fr_status_gpio tf_prefix="${tf_prefix}"/>
